Commit message: added lqr controller

File: src/diablo_env_ros/urdf/robot.urdf (robot description, URDF)
Before this commit: robot diablo, 16 links, 15 joints
Links:
- link left_leg_1: geometry visual mesh filename=file:///home/basanta-joshi/Desktop/virtual_environment/diab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
- link left_leg_2: geometry visual mesh filename=file:///home/basanta-joshi/Desktop/virtual_environment/diab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
- link left_leg_3: geometry collision box size=0.2 0.07 0.07; visual mesh filename=file:///home/basanta-joshi/Desktop/virtual_environment/diab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
- link right_leg_1: geometry visual mesh filename=file:///home/basanta-joshi/Desktop/virtual_environment/diab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
- link right_leg_2: geometry visual mesh filename=file:///home/basanta-joshi/Desktop/virtual_environment/diab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
- link right_leg_3: geometry collision box size=0.2 0.07 0.07; visual mesh filename=file:///home/basanta-joshi/Desktop/virtual_environment/diab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

File: src/diablo_env_ros/urdf/robot.xacro (robot description, xacro)
@@ -49,4 +49,6 @@
       <joint_name>joint_left_leg_2</joint_name>
       <joint_name>joint_right_leg_2</joint_name>
+      <joint_name>joint_left_leg_3</joint_name>
+      <joint_name>joint_right_leg_3</joint_name>
       <joint_name>joint_left_leg_4</joint_name>
       <joint_name>joint_right_leg_4</joint_name>
