Commit message: completely changed launch file and robot description along with gazebo tag including joint state joint controller

File: src/diablo_env_ros/urdf/description.xacro (robot description, xacro)
@@ -2,4 +2,5 @@
 <robot xmlns:xacro="http://www.ros.org/wiki/xacro" name="tita">
   <xacro:macro name="description">
+    <link name="world"/>
     <link name="base_link">
       <inertial>
@@ -22,7 +23,13 @@
       </collision>
     </link>
+    <joint name="base_link_joint" type="fixed">
+      <origin rpy="0 0 0" xyz="0 0 0.35"/>
+      <parent link="world"/>
+      <child link="base_link"/>
+      <axis xyz="0 0 0"/>
+    </joint>
     <link name="spad">
     </link>
-    <joint name="spad" type="fixed">
+    <joint name="joint_spad" type="fixed">
       <origin xyz="0.24052 -0.0019 0.064455" rpy="2.199 0 1.5708" />
       <parent link="base_link" />
@@ -32,5 +39,5 @@
     <link name="spad1">
     </link>
-    <joint name="spad1" type="fixed">
+    <joint name="joint_spad1" type="fixed">
       <origin xyz="0.21953 -0.0019 -0.030142" rpy="2.632 0 1.5708" />
       <parent link="base_link" />
@@ -40,5 +47,5 @@
     <link name="left_camera">
     </link>
-    <joint name="left_camera" type="fixed">
+    <joint name="joint_left_camera" type="fixed">
       <origin xyz="0.23416 0.075 0.04036" rpy="1.5708 0 1.5708" />
       <parent link="base_link" />
@@ -48,5 +55,5 @@
     <link name="ch201">
     </link>
-    <joint name="ch201" type="fixed">
+    <joint name="joint_ch201" type="fixed">
       <origin xyz="0.23782 0 0.018636" rpy="1.1693 0 1.5708" />
       <parent link="base_link" />
@@ -56,5 +63,5 @@
     <link name="right_camara">
     </link>
-    <joint name="right_camera" type="fixed">
+    <joint name="joint_right_camera" type="fixed">
       <origin xyz="0.23416 -0.075001 0.04036" rpy="1.5708 0 1.5708" />
       <parent link="base_link" />
@@ -62,4 +69,24 @@
       <axis xyz="0 0 0" />
     </joint>
+    <link name="imu_link">
+      <inertial>
+        <mass value="0.001"/>
+        <origin rpy="0 0 0" xyz="0 0 0"/>
+        <inertia ixx="0.0001" ixy="0" ixz="0" iyy="0.0001" iyz="0" izz="0.0001"/>
+      </inertial>
+      <visual>
+        <origin rpy="0 0 0" xyz="0 0 0"/>
+        <geometry>
+          <box size="0.001 0.001 0.001"/>
+        </geometry>
+        <material name="red"/>
+      </visual>
+      <collision>
+        <origin rpy="0 0 0" xyz="0 0 0"/>
+        <geometry>
+          <box size=".001 .001 .001"/>
+        </geometry>
+      </collision>
+    </link>
     <joint name="imu_joint" type="fixed">
       <parent link="base_link"/>
@@ -67,24 +94,4 @@
       <origin rpy="0 0 0" xyz="0 0 0"/>
     </joint>
-    <link name="imu_link">
-      <inertial>
-        <mass value="0.001"/>
-        <origin rpy="0 0 0" xyz="0 0 0"/>
-        <inertia ixx="0.0001" ixy="0" ixz="0" iyy="0.0001" iyz="0" izz="0.0001"/>
-      </inertial>
-      <visual>
-        <origin rpy="0 0 0" xyz="0 0 0"/>
-        <geometry>
-          <box size="0.001 0.001 0.001"/>
-        </geometry>
-        <material name="red"/>
-      </visual>
-      <collision>
-        <origin rpy="0 0 0" xyz="0 0 0"/>
-        <geometry>
-          <box size=".001 .001 .001"/>
-        </geometry>
-      </collision>
-    </link>
     <link name="left_leg_1">
       <inertial>
@@ -98,5 +105,5 @@
           <mesh filename="file://$(find diablo_env_ros)/meshes/left_leg_1.STL" />
         </geometry>
-        <material name="black"/>
+        <material name="blue"/>
       </visual>
     </link>
@@ -119,5 +126,5 @@
           <mesh filename="file://$(find diablo_env_ros)/meshes/left_leg_2.STL" />
         </geometry>
-        <material name="black"/>
+        <material name="green"/>
       </visual>
     </link>
@@ -140,5 +147,5 @@
           <mesh filename="file://$(find diablo_env_ros)/meshes/left_leg_3.STL" />
         </geometry>
-        <material name="black"/>
+        <material name="grey"/>
       </visual>
       <collision>
@@ -167,5 +174,5 @@
           <mesh filename="file://$(find diablo_env_ros)/meshes/left_leg_4.STL" />
         </geometry>
-        <material name="black"/>
+        <material name="silver"/>
       </visual>
       <collision>
@@ -194,5 +201,5 @@
           <mesh filename="file://$(find diablo_env_ros)/meshes/right_leg_1.STL" />
         </geometry>
-        <material name="black"/>
+        <material name="blue"/>
       </visual>
     </link>
@@ -215,5 +222,5 @@
           <mesh filename="file://$(find diablo_env_ros)/meshes/right_leg_2.STL" />
         </geometry>
-        <material name="black"/>
+        <material name="green"/>
       </visual>
     </link>
@@ -236,5 +243,5 @@
           <mesh filename="file://$(find diablo_env_ros)/meshes/right_leg_3.STL" />
         </geometry>
-        <material name="black"/>
+        <material name="grey"/>
       </visual>
       <collision>
@@ -263,5 +270,5 @@
           <mesh filename="file://$(find diablo_env_ros)/meshes/right_leg_4.STL" />
         </geometry>
-        <material name="black"/>
+        <material name="silver"/>
       </visual>
       <collision>

File: src/diablo_env_ros/urdf/robot.urdf (robot description, URDF)
Before this commit: robot tita, 15 links, 14 joints
Links:
- added link world
- link base_link: geometry collision box size=0.47 0.3 0.19; visual mesh filename=file:///home/basanta-joshi/Desktop/virtual_environment/diab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
- link ch201: mass 0.001 -> None
- link left_camera: mass 0.001 -> None
- link left_leg_1: geometry visual mesh filename=file:///home/basanta-joshi/Desktop/virtual_environment/diab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
- link left_leg_2: geometry visual mesh filename=file:///home/basanta-joshi/Desktop/virtual_environment/diab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
- link left_leg_3: geometry collision box size=0.2 0.07 0.05; visual mesh filename=file:///home/basanta-joshi/Desktop/virtual_environment/diab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
- link left_leg_4: geometry collision cylinder length=0.034 radius=0.0925; visual mesh filename=file:///home/basanta-joshi/Desktop/virtual_environment/diab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
- link right_camara: mass 0.001 -> None
- link right_leg_1: geometry visual mesh filename=file:///home/basanta-joshi/Desktop/virtual_environment/diab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
- link right_leg_2: geometry visual mesh filename=file:///home/basanta-joshi/Desktop/virtual_environment/diab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
- link right_leg_3: geometry collision box size=0.2 0.07 0.05; visual mesh filename=file:///home/basanta-joshi/Desktop/virtual_environment/diab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
- link right_leg_4: geometry collision cylinder length=0.034 radius=0.0925; visual mesh filename=file:///home/basanta-joshi/Desktop/virtual_environment/diab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
- link spad: mass 0.001 -> None
- link spad1: mass 0.001 -> None
Joints:
- removed joint ch201_joint
- removed joint left_camera_joint
- removed joint right_camera_joint
- removed joint spad1_joint
- removed joint spad_joint
- added joint base_link_joint: type fixed, parent world, child base_link, origin xyz=0 0 0.35 rpy=0 0 0, axis 0 0 0
- added joint joint_ch201: type fixed, parent base_link, child ch201, origin xyz=0.23782 0 0.018636 rpy=1.1693 0 1.5708, axis 0 0 0
- added joint joint_left_camera: type fixed, parent base_link, child left_camera, origin xyz=0.23416 0.075 0.04036 rpy=1.5708 0 1.5708, axis 0 0 0
- added joint joint_right_camera: type fixed, parent base_link, child right_camara, origin xyz=0.23416 -0.075001 0.04036 rpy=1.5708 0 1.5708, axis 0 0 0
- added joint joint_spad: type fixed, parent base_link, child spad, origin xyz=0.24052 -0.0019 0.064455 rpy=2.199 0 1.5708, axis 0 0 0
- added joint joint_spad1: type fixed, parent base_link, child spad1, origin xyz=0.21953 -0.0019 -0.030142 rpy=2.632 0 1.5708, axis 0 0 0

File: src/diablo_env_ros/urdf/robot.xacro (robot description, xacro)
@@ -1,4 +1,4 @@
 <?xml version="1.0"?>
-<robot xmlns:xacro="http://wiki.ros.org/xacro" name="tita">
+<robot xmlns:xacro="http://www.ros.org/xacro" name="diablo">
   <xacro:arg name="prefix" default="" />
   <xacro:arg name="use_tower" default="false" />
@@ -8,26 +8,33 @@
   <xacro:include filename="$(find diablo_env_ros)/urdf/materials.xacro" />
   <xacro:include filename="$(find diablo_env_ros)/urdf/description.xacro" />
-  <xacro:include filename="$(find diablo_env_ros)/urdf/ros2control.xacro" />
-  <xacro:include filename="$(find diablo_env_ros)/urdf/robot.gazebo" />
-  <xacro:ros2control name="diablo" ctrl_mode="position" sim_env="gazebo" yaml_path="$(find diablo_description)/config/controllers.yaml"/>
-  <xacro:if value="$(arg use_tower)">
-    <xacro:include filename="$(find diablo_env_ros)/urdf/tower.urdf.xacro" />
-    <joint name="tower_joint" type="fixed">
-      <parent link="base_link" />
-      <child link="tower_base_link" />
-      <origin xyz="0.0 0.0 0.1" rpy="0.0 0.0 0.0" />
-    </joint>
-    <xacro:tita_tower />
-  </xacro:if>
-  <xacro:if value="${sim_env == 'none'}">
-    <xacro:property name="name" value="HardwareControl" />
-  </xacro:if>
-  <xacro:if value="${sim_env == 'gazebo'}">
-    <xacro:property name="name" value="GazeboControl" />
-  </xacro:if>
-  <xacro:if value="${sim_env == 'webots'}">
-    <xacro:property name="name" value="WebotsControl" />
-  </xacro:if>
   <xacro:description />
-  <xacro:ros2control name="${name}" ctrl_mode="$(arg ctrl_mode)" sim_env="$(arg sim_env)" yaml_path="$(arg yaml_path)" />
+  <!-- Gazebo Physics Properties -->
+  <gazebo>
+    <mu1>0.5</mu1>       <!-- static friction coefficient -->
+    <mu2>0.3</mu2>       <!-- dynamic friction coefficient -->
+  </gazebo>
+  <!-- Gazebo Plugins and Sensors -->
+  <gazebo>
+    <plugin filename="gz-sim-joint-controller-system" name="gz::sim::systems::JointController">
+      <joint_name>joint_left_leg_1</joint_name>
+      <joint_name>joint_right_leg_1</joint_name>
+      <joint_name>joint_left_leg_2</joint_name>
+      <joint_name>joint_right_leg_2</joint_name>
+      <joint_name>joint_left_leg_4</joint_name>
+      <joint_name>joint_right_leg_4</joint_name>
+      <use_force_commands>true</use_force_commands>
+      <topic>effort_cmd</topic>
+    </plugin>
+    <plugin filename="gz-sim-joint-state-publisher-system" name="gz::sim::systems::JointStatePublisher">
+      <topic>joint_states</topic>
+      <joint_name>joint_left_leg_1</joint_name>
+      <joint_name>joint_right_leg_1</joint_name>
+      <joint_name>joint_left_leg_2</joint_name>
+      <joint_name>joint_right_leg_2</joint_name>
+      <joint_name>joint_left_leg_3</joint_name>
+      <joint_name>joint_right_leg_3</joint_name>
+      <joint_name>joint_left_leg_4</joint_name>
+      <joint_name>joint_right_leg_4</joint_name>
+    </plugin>
+  </gazebo>
 </robot>

Commit message: base_node

File: src/diablo_env_ros/urdf/description.xacro (robot description, xacro)
@@ -24,5 +24,5 @@
     </link>
     <joint name="base_link_joint" type="fixed">
-      <origin rpy="0 0 0" xyz="0 0 0.35"/>
+      <origin rpy="0 0 0" xyz="0 0 0.45"/>
       <parent link="world"/>
       <child link="base_link"/>
@@ -107,4 +107,10 @@
         <material name="blue"/>
       </visual>
+      <!-- <collision>
+        <origin xyz="0 0 0" rpy="0 0 0" />
+        <geometry>
+          <cylinder radius="0.035" length="0.1426" />
+        </geometry>
+      </collision> -->
     </link>
     <joint name="joint_left_leg_1" type="revolute">
@@ -128,4 +134,10 @@
         <material name="green"/>
       </visual>
+      <!-- <collision>
+        <origin xyz="-0.1426 0 0" rpy="1.5708 0 1.5708" />
+        <geometry>
+          <cylinder radius="0.035" length="0.2" />
+        </geometry>
+      </collision> -->
     </link>
     <joint name="joint_left_leg_2" type="revolute">
@@ -152,5 +164,5 @@
         <origin xyz="0.1 0.021 -0.002" rpy="0 0 -0.131" />
         <geometry>
-          <box size="0.2 0.07 0.05" />
+          <box size="0.2 0.07 0.07" />
         </geometry>
       </collision>
@@ -203,4 +215,10 @@
         <material name="blue"/>
       </visual>
+      <!-- <collision>
+        <origin xyz="0 0 0" rpy="0 0 0" />
+        <geometry>
+          <cylinder radius="0.035" length="0.1426" />
+        </geometry>
+      </collision> -->
     </link>
     <joint name="joint_right_leg_1" type="revolute">
@@ -224,4 +242,10 @@
         <material name="green"/>
       </visual>
+      <!-- <collision>
+        <origin xyz="-0.1426 0 0" rpy="1.5708 0 1.5708" />
+        <geometry>
+          <cylinder radius="0.035" length="0.2" />
+        </geometry>
+      </collision> -->
     </link>
     <joint name="joint_right_leg_2" type="revolute">
@@ -248,5 +272,5 @@
         <origin xyz="0.1 0.021 -0.002" rpy="0 0 -0.131" />
         <geometry>
-          <box size="0.2 0.07 0.05" />
+          <box size="0.2 0.07 0.07" />
         </geometry>
       </collision>

File: src/diablo_env_ros/urdf/robot.urdf (robot description, URDF)
Before this commit: robot diablo, 16 links, 15 joints
Links:
- link left_leg_1: geometry collision cylinder length=0.1426 radius=0.035; visual mesh filename=file:///home/basanta-joshi/Desktop/virtual_environment/diab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
- link left_leg_2: geometry collision cylinder length=0.2 radius=0.035; visual mesh filename=file:///home/basanta-joshi/Desktop/virtual_environment/diab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
- link left_leg_3: geometry collision cylinder length=0.2 radius=0.35; visual mesh filename=file:///home/basanta-joshi/Desktop/virtual_environment/diab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
- link right_leg_1: geometry collision cylinder length=0.1426 radius=0.035; visual mesh filename=file:///home/basanta-joshi/Desktop/virtual_environment/diab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
- link right_leg_2: geometry collision cylinder length=0.2 radius=0.035; visual mesh filename=file:///home/basanta-joshi/Desktop/virtual_environment/diab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
- link right_leg_3: geometry collision cylinder length=0.2 radius=0.035; visual mesh filename=file:///home/basanta-joshi/Desktop/virtual_environment/diab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
Joints:
- joint base_link_joint: origin xyz=0 0 0.35 rpy=0 0 0 -> xyz=0 0 0.45 rpy=0 0 0

File: src/diablo_env_ros/urdf/robot.xacro (robot description, xacro)
@@ -13,4 +13,32 @@
     <mu1>0.5</mu1>       <!-- static friction coefficient -->
     <mu2>0.3</mu2>       <!-- dynamic friction coefficient -->
+  </gazebo>
+  <!-- Enable Self-Collisions -->
+  <gazebo reference="base_link">
+    <self_collide>true</self_collide>
+  </gazebo>
+  <gazebo reference="left_leg_1">
+    <self_collide>true</self_collide>
+  </gazebo>
+  <gazebo reference="left_leg_2">
+    <self_collide>true</self_collide>
+  </gazebo>
+  <gazebo reference="left_leg_3">
+    <self_collide>true</self_collide>
+  </gazebo>
+  <gazebo reference="left_leg_4">
+    <self_collide>true</self_collide>
+  </gazebo>
+  <gazebo reference="right_leg_1">
+    <self_collide>true</self_collide>
+  </gazebo>
+  <gazebo reference="right_leg_2">
+    <self_collide>true</self_collide>
+  </gazebo>
+  <gazebo reference="right_leg_3">
+    <self_collide>true</self_collide>
+  </gazebo>
+  <gazebo reference="right_leg_4">
+    <self_collide>true</self_collide>
   </gazebo>
   <!-- Gazebo Plugins and Sensors -->

Commit message: check

File: src/diablo_env_ros/urdf/description.xacro (robot description, xacro)
@@ -24,5 +24,5 @@
     </link>
     <joint name="base_link_joint" type="fixed">
-      <origin rpy="0 0 0" xyz="0 0 0.45"/>
+      <origin rpy="0 0 0" xyz="0 0 0.35"/>
       <parent link="world"/>
       <child link="base_link"/>

Commit message: added imu

File: src/diablo_env_ros/urdf/description.xacro (robot description, xacro)
@@ -2,5 +2,5 @@
 <robot xmlns:xacro="http://www.ros.org/wiki/xacro" name="tita">
   <xacro:macro name="description">
-    <link name="world"/>
+    <!-- <link name="world"/> -->
     <link name="base_link">
       <inertial>
@@ -17,16 +17,16 @@
       </visual>
       <collision>
-        <origin xyz="0 0 0.017" rpy="0 0 0" />
-        <geometry>
-          <box size="0.47 0.3 0.19" />
-        </geometry>
-      </collision>
-    </link>
-    <joint name="base_link_joint" type="fixed">
-      <origin rpy="0 0 0" xyz="0 0 0.35"/>
+        <origin xyz="0 0 0" rpy="0 0 0" />
+        <geometry>
+          <mesh filename="file://$(find diablo_env_ros)/meshes/base_link.STL" />
+        </geometry>
+      </collision>
+    </link>
+    <!-- <joint name="base_link_joint" type="fixed">
+      <origin rpy="0 0 0" xyz="0 0 0.41"/>
       <parent link="world"/>
       <child link="base_link"/>
       <axis xyz="0 0 0"/>
-    </joint>
+    </joint> -->
     <link name="spad">
     </link>
@@ -107,10 +107,10 @@
         <material name="blue"/>
       </visual>
-      <!-- <collision>
-        <origin xyz="0 0 0" rpy="0 0 0" />
-        <geometry>
-          <cylinder radius="0.035" length="0.1426" />
-        </geometry>
-      </collision> -->
+      <collision>
+        <origin xyz="0 0 0" rpy="0 0 0" />
+        <geometry>
+          <mesh filename="file://$(find diablo_env_ros)/meshes/left_leg_1.STL" />
+        </geometry>
+      </collision>
     </link>
     <joint name="joint_left_leg_1" type="revolute">
@@ -134,10 +134,10 @@
         <material name="green"/>
       </visual>
-      <!-- <collision>
-        <origin xyz="-0.1426 0 0" rpy="1.5708 0 1.5708" />
-        <geometry>
-          <cylinder radius="0.035" length="0.2" />
-        </geometry>
-      </collision> -->
+      <collision>
+        <origin xyz="0 0 0" rpy="0 0 0" />
+        <geometry>
+          <mesh filename="file://$(find diablo_env_ros)/meshes/left_leg_2.STL" />
+        </geometry>
+      </collision>
     </link>
     <joint name="joint_left_leg_2" type="revolute">
@@ -162,7 +162,7 @@
       </visual>
       <collision>
-        <origin xyz="0.1 0.021 -0.002" rpy="0 0 -0.131" />
-        <geometry>
-          <box size="0.2 0.07 0.07" />
+        <origin xyz="0 0 0" rpy="0 0 0" />
+        <geometry>
+          <mesh filename="file://$(find diablo_env_ros)/meshes/left_leg_3.STL" />
         </geometry>
       </collision>
@@ -191,5 +191,5 @@
         <origin xyz="0 0 0" rpy="0 0 0" />
         <geometry>
-          <cylinder radius="0.0925" length="0.034" />
+          <mesh filename="file://$(find diablo_env_ros)/meshes/left_leg_4.STL" />
         </geometry>
       </collision>
@@ -215,10 +215,10 @@
         <material name="blue"/>
       </visual>
-      <!-- <collision>
-        <origin xyz="0 0 0" rpy="0 0 0" />
-        <geometry>
-          <cylinder radius="0.035" length="0.1426" />
-        </geometry>
-      </collision> -->
+      <collision>
+        <origin xyz="0 0 0" rpy="0 0 0" />
+        <geometry>
+          <mesh filename="file://$(find diablo_env_ros)/meshes/right_leg_1.STL" />
+        </geometry>
+      </collision>
     </link>
     <joint name="joint_right_leg_1" type="revolute">
@@ -242,10 +242,10 @@
         <material name="green"/>
       </visual>
-      <!-- <collision>
-        <origin xyz="-0.1426 0 0" rpy="1.5708 0 1.5708" />
-        <geometry>
-          <cylinder radius="0.035" length="0.2" />
-        </geometry>
-      </collision> -->
+      <collision>
+        <origin xyz="0 0 0" rpy="0 0 0" />
+        <geometry>
+          <mesh filename="file://$(find diablo_env_ros)/meshes/right_leg_2.STL" />
+        </geometry>
+      </collision>
     </link>
     <joint name="joint_right_leg_2" type="revolute">
@@ -270,7 +270,7 @@
       </visual>
       <collision>
-        <origin xyz="0.1 0.021 -0.002" rpy="0 0 -0.131" />
-        <geometry>
-          <box size="0.2 0.07 0.07" />
+        <origin xyz="0 0 0" rpy="0 0 0" />
+        <geometry>
+          <mesh filename="file://$(find diablo_env_ros)/meshes/right_leg_3.STL" />
         </geometry>
       </collision>
@@ -299,5 +299,5 @@
         <origin xyz="0 0 0" rpy="0 0 0" />
         <geometry>
-          <cylinder radius="0.0925" length="0.034" />
+          <mesh filename="file://$(find diablo_env_ros)/meshes/right_leg_4.STL" />
         </geometry>
       </collision>

File: src/diablo_env_ros/urdf/robot.urdf (robot description, URDF)
Before this commit: robot diablo, 16 links, 15 joints
Links:
- removed link world
- link base_link: geometry collision mesh filename=file:///home/basanta-joshi/Desktop/virtual_environment/diab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; visual mesh filename=file:///home/basanta-joshi/Desktop/virtual_environment/diab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
- link left_leg_1: geometry collision mesh filename=file:///home/basanta-joshi/Desktop/virtual_environment/diab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; visual mesh filename=file:///home/basanta-joshi/Desktop/virtual_environment/diab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
- link left_leg_2: geometry collision mesh filename=file:///home/basanta-joshi/Desktop/virtual_environment/diab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; visual mesh filename=file:///home/basanta-joshi/Desktop/virtual_environment/diab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
- link left_leg_3: geometry collision mesh filename=file:///home/basanta-joshi/Desktop/virtual_environment/diab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; visual mesh filename=file:///home/basanta-joshi/Desktop/virtual_environment/diab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
- link left_leg_4: geometry collision mesh filename=file:///home/basanta-joshi/Desktop/virtual_environment/diab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; visual mesh filename=file:///home/basanta-joshi/Desktop/virtual_environment/diab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
- link right_leg_1: geometry collision mesh filename=file:///home/basanta-joshi/Desktop/virtual_environment/diab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; visual mesh filename=file:///home/basanta-joshi/Desktop/virtual_environment/diab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
- link right_leg_2: geometry collision mesh filename=file:///home/basanta-joshi/Desktop/virtual_environment/diab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; visual mesh filename=file:///home/basanta-joshi/Desktop/virtual_environment/diab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
- link right_leg_3: geometry collision mesh filename=file:///home/basanta-joshi/Desktop/virtual_environment/diab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; visual mesh filename=file:///home/basanta-joshi/Desktop/virtual_environment/diab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
- link right_leg_4: geometry collision mesh filename=file:///home/basanta-joshi/Desktop/virtual_environment/diab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; visual mesh filename=file:///home/basanta-joshi/Desktop/virtual_environment/diab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
Joints:
- removed joint base_link_joint

File: src/diablo_env_ros/urdf/robot.xacro (robot description, xacro)
@@ -68,3 +68,13 @@
     </plugin>
   </gazebo>
+  <gazebo reference="imu_link">
+    <sensor name="imu" type="imu">
+      <always_on>1</always_on>
+      <update_rate>50</update_rate>
+      <visualize>true</visualize>
+      <topic>imu</topic>
+      <enable_metrics>true</enable_metrics>
+      <gz_frame_id>imu_link</gz_frame_id>
+    </sensor>
+  </gazebo>
 </robot>
