Commit message: added lidar

File: src/diablo_env_ros/urdf/description.xacro (robot description, xacro)
@@ -3,4 +3,11 @@
   <xacro:macro name="description">
     <!-- <link name="world"/> -->
+    <link name="base_footprint">
+      <inertial>
+        <mass value="0.0001"/>
+        <origin xyz="0 0 0" rpy="0 0 0"/>
+        <inertia ixx="1e-6" ixy="0" ixz="0" iyy="1e-6" iyz="0" izz="1e-6"/>
+      </inertial>
+    </link>
     <link name="base_link">
       <inertial>
@@ -29,4 +36,33 @@
       <axis xyz="0 0 0"/>
     </joint> -->
+    <joint name="base_footprint_joint" type="fixed">
+      <parent link="base_footprint"/>
+      <child link="base_link"/>
+      <origin xyz="0 0 0.4925" rpy="0 0 0"/>
+    </joint>
+    <link name="down_lidar_link">
+      <visual>
+        <origin rpy="0 0 0" xyz="0 0 0"/>
+        <geometry>
+          <box size="0.01 0.01 0.01"/>
+        </geometry>
+        <material name="green"/>
+      </visual>
+      <collision>
+        <origin rpy="0 0 0" xyz="0 0 0"/>
+        <geometry>
+          <box size="0.01 0.01 0.01"/>
+        </geometry>
+      </collision>
+      <inertial>
+        <mass value="0.001"/>
+        <inertia ixx="0.00001" ixy="0.0" ixz="0.0" iyy="0.00001" iyz="0.0" izz="0.00001"/>
+      </inertial>
+    </link>
+    <joint name="down_lidar_joint" type="fixed">
+      <parent link="base_link"/>      <!-- or whichever link is below -->
+      <child link="down_lidar_link"/>
+      <origin xyz="0 0 0.3" rpy="0 1.5708 0"/> <!-- adjust height so it’s just below robot -->
+    </joint>
     <link name="spad">
     </link>

File: src/diablo_env_ros/urdf/robot.urdf (robot description, URDF)
Before this commit: robot diablo, 15 links, 14 joints
Links:
- added link base_footprint, mass 0.0001
- added link down_lidar_link, mass 0.001; collision box size=0.01 0.01 0.01; visual box size=0.01 0.01 0.01
Joints:
- added joint base_footprint_joint: type fixed, parent base_footprint, child base_link, origin xyz=0 0 0.4925 rpy=0 0 0
- added joint down_lidar_joint: type fixed, parent base_link, child down_lidar_link, origin xyz=0 0 0.3 rpy=0 1.5708 0

File: src/diablo_env_ros/urdf/robot.xacro (robot description, xacro)
@@ -78,3 +78,35 @@
     </sensor>
   </gazebo>
+  <gazebo reference="down_lidar_link">
+    <sensor name="down_lidar" type="ray">
+      <pose>0 0 0 0 0 0</pose>
+      <ray>
+        <scan>
+          <horizontal>
+            <samples>1</samples>
+            <resolution>1</resolution>
+            <min_angle>0</min_angle>
+            <max_angle>0</max_angle>
+          </horizontal>
+          <vertical>
+            <samples>1</samples>
+            <resolution>1</resolution>
+            <min_angle>-1.5708</min_angle>  <!-- Pointing straight down -->
+            <max_angle>-1.5708</max_angle>
+          </vertical>
+        </scan>
+        <range>
+          <min>0.05</min>
+          <max>5.0</max>
+          <resolution>0.01</resolution>
+        </range>
+      </ray>
+      <always_on>true</always_on>
+      <update_rate>20</update_rate>
+      <visualize>true</visualize>
+      <plugin filename="libgz-sim-sensors-system.so" name="gz::sim::systems::Sensors">
+        <topic>/down_lidar</topic>
+      </plugin>
+    </sensor>
+  </gazebo>
 </robot>

Commit message: added 3d lidar instead of rangefinder

File: src/diablo_env_ros/urdf/description.xacro (robot description, xacro)
@@ -41,5 +41,5 @@
       <origin xyz="0 0 0.4925" rpy="0 0 0"/>
     </joint>
-    <link name="down_lidar_link">
+    <link name="lidar_frame">
       <visual>
         <origin rpy="0 0 0" xyz="0 0 0"/>
@@ -60,8 +60,8 @@
       </inertial>
     </link>
-    <joint name="down_lidar_joint" type="fixed">
+    <joint name="lidar_frame_joint" type="fixed">
       <parent link="base_link"/>      <!-- or whichever link is below -->
-      <child link="down_lidar_link"/>
-      <origin xyz="0 0 0.3" rpy="0 1.5708 0"/> <!-- adjust height so it’s just below robot -->
+      <child link="lidar_frame"/>
+      <origin xyz="0 0 0" rpy="0 1.5708 0"/> <!-- adjust height so it’s just below robot -->
     </joint>
     <link name="spad">
@@ -155,5 +155,5 @@
       <child link="left_leg_1" />
       <axis xyz="0 0 1" />
-      <limit lower="-0.785398" upper="0.785398" effort="100" velocity="100" />
+      <limit lower="-0.1" upper="0.1" effort="100" velocity="100" />
     </joint>
     <link name="left_leg_2">
@@ -263,5 +263,5 @@
       <child link="right_leg_1" />
       <axis xyz="0 0 1" />
-      <limit lower="-0.785398" upper="0.785398" effort="100" velocity="100" />
+      <limit lower="-0.1" upper="0.1" effort="100" velocity="100" />
     </joint>
     <link name="right_leg_2">

File: src/diablo_env_ros/urdf/robot.urdf (robot description, URDF)
Before this commit: robot diablo, 17 links, 16 joints
Links:
- removed link down_lidar_link
- added link lidar_frame, mass 0.001; collision box size=0.01 0.01 0.01; visual box size=0.01 0.01 0.01
Joints:
- removed joint down_lidar_joint
- added joint lidar_frame_joint: type fixed, parent base_link, child lidar_frame, origin xyz=0 0 0 rpy=0 1.5708 0
- joint joint_left_leg_1: limit lower=-0.785398 upper=0.785398 effort=100 velocity=100 -> lower=-0.1 upper=0.1 effort=100 velocity=100
- joint joint_right_leg_1: limit lower=-0.785398 upper=0.785398 effort=100 velocity=100 -> lower=-0.1 upper=0.1 effort=100 velocity=100

File: src/diablo_env_ros/urdf/robot.xacro (robot description, xacro)
@@ -78,34 +78,27 @@
     </sensor>
   </gazebo>
-  <gazebo reference="down_lidar_link">
-    <sensor name="down_lidar" type="ray">
-      <pose>0 0 0 0 0 0</pose>
-      <ray>
-        <scan>
-          <horizontal>
-            <samples>1</samples>
-            <resolution>1</resolution>
-            <min_angle>0</min_angle>
-            <max_angle>0</max_angle>
-          </horizontal>
-          <vertical>
-            <samples>1</samples>
-            <resolution>1</resolution>
-            <min_angle>-1.5708</min_angle>  <!-- Pointing straight down -->
-            <max_angle>-1.5708</max_angle>
-          </vertical>
-        </scan>
-        <range>
-          <min>0.05</min>
-          <max>5.0</max>
-          <resolution>0.01</resolution>
-        </range>
-      </ray>
-      <always_on>true</always_on>
-      <update_rate>20</update_rate>
-      <visualize>true</visualize>
-      <plugin filename="libgz-sim-sensors-system.so" name="gz::sim::systems::Sensors">
-        <topic>/down_lidar</topic>
-      </plugin>
+  <gazebo reference="lidar_frame">
+    <sensor name='gpu_lidar' type='gpu_lidar'>"
+        <pose relative_to='lidar_frame'>0 0 0 0 0 0</pose>
+        <topic>lidar</topic>
+        <gz_frame_id>lidar_frame</gz_frame_id>
+        <update_rate>10</update_rate>
+        <ray>
+            <scan>
+                <horizontal>
+                    <samples>3</samples>
+                    <resolution>1</resolution>
+                    <min_angle>-1.5708</min_angle>
+                    <max_angle>1.5708</max_angle>
+                </horizontal>
+            </scan>
+            <range>
+                <min>0.08</min>
+                <max>10.0</max>
+                <resolution>0.01</resolution>
+            </range>
+        </ray>
+        <always_on>1</always_on>
+        <visualize>true</visualize>
     </sensor>
   </gazebo>

Commit message: there was a mismatch in topic publishing and subscribing in joint torques and collision was also changes as gazebo was showing ode solving error

File: src/diablo_env_ros/urdf/description.xacro (robot description, xacro)
@@ -26,5 +26,6 @@
         <origin xyz="0 0 0" rpy="0 0 0" />
         <geometry>
-          <mesh filename="file://$(find diablo_env_ros)/meshes/base_link.STL" />
+          <box size="0.47 0.3 0.19"/>
+          <!-- <mesh filename="file://$(find diablo_env_ros)/meshes/base_link.STL" /> -->
         </geometry>
       </collision>
@@ -49,10 +50,10 @@
         <material name="green"/>
       </visual>
-      <collision>
+      <!-- <collision>
         <origin rpy="0 0 0" xyz="0 0 0"/>
         <geometry>
           <box size="0.01 0.01 0.01"/>
         </geometry>
-      </collision>
+      </collision> -->
       <inertial>
         <mass value="0.001"/>
@@ -118,10 +119,10 @@
         <material name="red"/>
       </visual>
-      <collision>
+      <!-- <collision>
         <origin rpy="0 0 0" xyz="0 0 0"/>
         <geometry>
           <box size=".001 .001 .001"/>
         </geometry>
-      </collision>
+      </collision> -->
     </link>
     <joint name="imu_joint" type="fixed">
@@ -143,10 +144,10 @@
         <material name="blue"/>
       </visual>
-      <collision>
+      <!-- <collision>
         <origin xyz="0 0 0" rpy="0 0 0" />
         <geometry>
           <mesh filename="file://$(find diablo_env_ros)/meshes/left_leg_1.STL" />
         </geometry>
-      </collision>
+      </collision> -->
     </link>
     <joint name="joint_left_leg_1" type="revolute">
@@ -170,10 +171,10 @@
         <material name="green"/>
       </visual>
-      <collision>
+      <!-- <collision>
         <origin xyz="0 0 0" rpy="0 0 0" />
         <geometry>
           <mesh filename="file://$(find diablo_env_ros)/meshes/left_leg_2.STL" />
         </geometry>
-      </collision>
+      </collision> -->
     </link>
     <joint name="joint_left_leg_2" type="revolute">
@@ -198,7 +199,8 @@
       </visual>
       <collision>
-        <origin xyz="0 0 0" rpy="0 0 0" />
-        <geometry>
-          <mesh filename="file://$(find diablo_env_ros)/meshes/left_leg_3.STL" />
+        <origin xyz="0.131 0 0" rpy="0 0 0" />
+        <geometry>
+          <box size="0.2 0.07 0.05"/>
+          <!-- <mesh filename="file://$(find diablo_env_ros)/meshes/left_leg_3.STL" /> -->
         </geometry>
       </collision>
@@ -220,4 +222,5 @@
         <origin xyz="0 0 0" rpy="0 0 0" />
         <geometry>
+          <!-- <cylinder length="0.034" radius="0.0925"/> -->
           <mesh filename="file://$(find diablo_env_ros)/meshes/left_leg_4.STL" />
         </geometry>
@@ -227,5 +230,6 @@
         <origin xyz="0 0 0" rpy="0 0 0" />
         <geometry>
-          <mesh filename="file://$(find diablo_env_ros)/meshes/left_leg_4.STL" />
+          <cylinder length="0.034" radius="0.0925"/>
+          <!-- <mesh filename="file://$(find diablo_env_ros)/meshes/left_leg_4.STL" /> -->
         </geometry>
       </collision>
@@ -251,10 +255,10 @@
         <material name="blue"/>
       </visual>
-      <collision>
+      <!-- <collision>
         <origin xyz="0 0 0" rpy="0 0 0" />
         <geometry>
           <mesh filename="file://$(find diablo_env_ros)/meshes/right_leg_1.STL" />
         </geometry>
-      </collision>
+      </collision> -->
     </link>
     <joint name="joint_right_leg_1" type="revolute">
@@ -278,10 +282,10 @@
         <material name="green"/>
       </visual>
-      <collision>
+      <!-- <collision>
         <origin xyz="0 0 0" rpy="0 0 0" />
         <geometry>
           <mesh filename="file://$(find diablo_env_ros)/meshes/right_leg_2.STL" />
         </geometry>
-      </collision>
+      </collision> -->
     </link>
     <joint name="joint_right_leg_2" type="revolute">
@@ -306,7 +310,8 @@
       </visual>
       <collision>
-        <origin xyz="0 0 0" rpy="0 0 0" />
-        <geometry>
-          <mesh filename="file://$(find diablo_env_ros)/meshes/right_leg_3.STL" />
+        <origin xyz="0.131 0 0" rpy="0 0 0" />
+        <geometry>
+          <box size="0.2 0.07 0.05"/>
+          <!-- <mesh filename="file://$(find diablo_env_ros)/meshes/right_leg_3.STL" /> -->
         </geometry>
       </collision>
@@ -335,5 +340,6 @@
         <origin xyz="0 0 0" rpy="0 0 0" />
         <geometry>
-          <mesh filename="file://$(find diablo_env_ros)/meshes/right_leg_4.STL" />
+          <cylinder length="0.034" radius="0.0925"/>
+          <!-- <mesh filename="file://$(find diablo_env_ros)/meshes/right_leg_4.STL" /> -->
         </geometry>
       </collision>

File: src/diablo_env_ros/urdf/robot.urdf (robot description, URDF)
Before this commit: robot diablo, 17 links, 16 joints
Links:
- link base_link: geometry collision box size=0.47 0.3 0.19; visual mesh filename=file:///home/basanta-joshi/Desktop/virtual_environment/diab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
- link imu_link: geometry visual box size=0.001 0.001 0.001
- link left_leg_1: geometry visual mesh filename=file:///home/basanta-joshi/Desktop/virtual_environment/diab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
- link left_leg_2: geometry visual mesh filename=file:///home/basanta-joshi/Desktop/virtual_environment/diab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
- link left_leg_3: geometry collision box size=0.2 0.07 0.05; visual mesh filename=file:///home/basanta-joshi/Desktop/virtual_environment/diab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
- link left_leg_4: geometry collision cylinder length=0.034 radius=0.0925; visual mesh filename=file:///home/basanta-joshi/Desktop/virtual_environment/diab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
- link lidar_frame: geometry visual box size=0.01 0.01 0.01
- link right_leg_1: geometry visual mesh filename=file:///home/basanta-joshi/Desktop/virtual_environment/diab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
- link right_leg_2: geometry visual mesh filename=file:///home/basanta-joshi/Desktop/virtual_environment/diab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
- link right_leg_3: geometry collision box size=0.2 0.07 0.05; visual mesh filename=file:///home/basanta-joshi/Desktop/virtual_environment/diab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
- link right_leg_4: geometry collision cylinder length=0.034 radius=0.0925; visual mesh filename=file:///home/basanta-joshi/Desktop/virtual_environment/diab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

File: src/diablo_env_ros/urdf/robot.xacro (robot description, xacro)
@@ -46,13 +46,41 @@
     <plugin filename="gz-sim-joint-controller-system" name="gz::sim::systems::JointController">
       <joint_name>joint_left_leg_1</joint_name>
+      <topic>joint_left_leg_1_effort</topic>
+      <use_force_commands>true</use_force_commands>
+    </plugin>
+    <plugin filename="gz-sim-joint-controller-system" name="gz::sim::systems::JointController">
       <joint_name>joint_right_leg_1</joint_name>
+      <topic>joint_right_leg_1_effort</topic>
+      <use_force_commands>true</use_force_commands>
+    </plugin>
+    <plugin filename="gz-sim-joint-controller-system" name="gz::sim::systems::JointController">
       <joint_name>joint_left_leg_2</joint_name>
+      <topic>joint_left_leg_2_effort</topic>
+      <use_force_commands>true</use_force_commands>
+    </plugin>
+    <plugin filename="gz-sim-joint-controller-system" name="gz::sim::systems::JointController">
       <joint_name>joint_right_leg_2</joint_name>
+      <topic>joint_right_leg_2_effort</topic>
+      <use_force_commands>true</use_force_commands>
+    </plugin>
+    <plugin filename="gz-sim-joint-controller-system" name="gz::sim::systems::JointController">
       <joint_name>joint_left_leg_3</joint_name>
+      <topic>joint_left_leg_3_effort</topic>
+      <use_force_commands>true</use_force_commands>
+    </plugin>
+    <plugin filename="gz-sim-joint-controller-system" name="gz::sim::systems::JointController">
       <joint_name>joint_right_leg_3</joint_name>
+      <topic>joint_right_leg_3_effort</topic>
+      <use_force_commands>true</use_force_commands>
+    </plugin>
+    <plugin filename="gz-sim-joint-controller-system" name="gz::sim::systems::JointController">
       <joint_name>joint_left_leg_4</joint_name>
+      <topic>joint_left_leg_4_effort</topic>
+      <use_force_commands>true</use_force_commands>
+    </plugin>
+    <plugin filename="gz-sim-joint-controller-system" name="gz::sim::systems::JointController">
       <joint_name>joint_right_leg_4</joint_name>
+      <topic>joint_right_leg_4_effort</topic>
       <use_force_commands>true</use_force_commands>
-      <topic>effort_cmd</topic>
     </plugin>
     <plugin filename="gz-sim-joint-state-publisher-system" name="gz::sim::systems::JointStatePublisher">

Commit message: new_launch_file for launching all three nodes for subscription simulation and learning with 2 second time delay

File: src/diablo_env_ros/urdf/description.xacro (robot description, xacro)
@@ -156,5 +156,5 @@
       <child link="left_leg_1" />
       <axis xyz="0 0 1" />
-      <limit lower="-0.1" upper="0.1" effort="100" velocity="100" />
+      <limit lower="-0.7854" upper="0.7854" effort="100" velocity="100" />
     </joint>
     <link name="left_leg_2">

File: src/diablo_env_ros/urdf/robot.urdf (robot description, URDF)
Before this commit: robot diablo, 17 links, 16 joints
Joints:
- joint joint_left_leg_1: limit lower=-0.1 upper=0.1 effort=100 velocity=100 -> lower=-0.7854 upper=0.7854 effort=100 velocity=100

Commit message: i need better reward system huhu

File: src/diablo_env_ros/urdf/description.xacro (robot description, xacro)
@@ -12,5 +12,5 @@
     <link name="base_link">
       <inertial>
-        <origin xyz="0.020452 3.5457E-06 0.01871" rpy="0 0 0" />
+        <origin xyz="-0.020452 3.5457E-06 0.01871" rpy="0 0 0" />
         <mass value="13.2" />
         <inertia ixx="0.061855" ixy="-2.6029E-05" ixz="0.00081082" iyy="0.036934" iyz="-1.7269E-05" izz="0.071232" />
@@ -26,5 +26,6 @@
         <origin xyz="0 0 0" rpy="0 0 0" />
         <geometry>
-          <box size="0.47 0.3 0.19"/>
+          <sphere radius="0.15"/>
+          <!-- <box size="0.47 0.3 0.19"/> -->
           <!-- <mesh filename="file://$(find diablo_env_ros)/meshes/base_link.STL" /> -->
         </geometry>
@@ -66,5 +67,5 @@
       <origin xyz="0 0 0" rpy="0 1.5708 0"/> <!-- adjust height so it’s just below robot -->
     </joint>
-    <link name="spad">
+    <!-- <link name="spad">
     </link>
     <joint name="joint_spad" type="fixed">
@@ -105,5 +106,5 @@
       <child link="right_camara" />
       <axis xyz="0 0 0" />
-    </joint>
+    </joint> -->
     <link name="imu_link">
       <inertial>
@@ -171,10 +172,11 @@
         <material name="green"/>
       </visual>
-      <!-- <collision>
-        <origin xyz="0 0 0" rpy="0 0 0" />
-        <geometry>
+      <collision>
+        <origin xyz="0.1 0 0" rpy="0 0 0" />
+        <geometry>
+          <box size="0.2 0.07 0.05"/>
           <mesh filename="file://$(find diablo_env_ros)/meshes/left_leg_2.STL" />
         </geometry>
-      </collision> -->
+      </collision>
     </link>
     <joint name="joint_left_leg_2" type="revolute">
@@ -282,10 +284,11 @@
         <material name="green"/>
       </visual>
-      <!-- <collision>
-        <origin xyz="0 0 0" rpy="0 0 0" />
-        <geometry>
+      <collision>
+        <origin xyz="0.1 0 0" rpy="0 0 0" />
+        <geometry>
+          <box size="0.2 0.07 0.05"/>
           <mesh filename="file://$(find diablo_env_ros)/meshes/right_leg_2.STL" />
         </geometry>
-      </collision> -->
+      </collision>
     </link>
     <joint name="joint_right_leg_2" type="revolute">

File: src/diablo_env_ros/urdf/robot.urdf (robot description, URDF)
Before this commit: robot diablo, 17 links, 16 joints
Links:
- removed link ch201
- removed link left_camera
- removed link right_camara
- removed link spad
- removed link spad1
- link base_link: geometry collision sphere radius=0.15; visual mesh filename=file:///home/basanta-joshi/Desktop/virtual_environment/diab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
- link left_leg_2: geometry collision box size=0.2 0.07 0.05; visual mesh filename=file:///home/basanta-joshi/Desktop/virtual_environment/diab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
- link right_leg_2: geometry collision box size=0.2 0.07 0.05; visual mesh filename=file:///home/basanta-joshi/Desktop/virtual_environment/diab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
Joints:
- removed joint joint_ch201
- removed joint joint_left_camera
- removed joint joint_right_camera
- removed joint joint_spad
- removed joint joint_spad1

Commit message: a2c milayeko alikati

File: src/diablo_env_ros/urdf/description.xacro (robot description, xacro)
@@ -224,6 +224,7 @@
         <origin xyz="0 0 0" rpy="0 0 0" />
         <geometry>
+          <box size="0.0925 0.0925 0.0925"/>
           <!-- <cylinder length="0.034" radius="0.0925"/> -->
-          <mesh filename="file://$(find diablo_env_ros)/meshes/left_leg_4.STL" />
+          <!-- <mesh filename="file://$(find diablo_env_ros)/meshes/left_leg_4.STL" /> -->
         </geometry>
         <material name="silver"/>
@@ -232,5 +233,6 @@
         <origin xyz="0 0 0" rpy="0 0 0" />
         <geometry>
-          <cylinder length="0.034" radius="0.0925"/>
+          <box size="0.0925 0.0925 0.0925"/>
+          <!-- <cylinder length="0.034" radius="0.0925"/> -->
           <!-- <mesh filename="file://$(find diablo_env_ros)/meshes/left_leg_4.STL" /> -->
         </geometry>
@@ -336,5 +338,6 @@
         <origin xyz="0 0 0" rpy="0 0 0" />
         <geometry>
-          <mesh filename="file://$(find diablo_env_ros)/meshes/right_leg_4.STL" />
+          <box size="0.0925 0.0925 0.0925"/>
+          <!-- <mesh filename="file://$(find diablo_env_ros)/meshes/right_leg_4.STL" /> -->
         </geometry>
         <material name="silver"/>
@@ -343,10 +346,11 @@
         <origin xyz="0 0 0" rpy="0 0 0" />
         <geometry>
-          <cylinder length="0.034" radius="0.0925"/>
+          <box size="0.0925 0.0925 0.0925"/>
+          <!-- <cylinder length="0.034" radius="0.0925"/> -->
           <!-- <mesh filename="file://$(find diablo_env_ros)/meshes/right_leg_4.STL" /> -->
         </geometry>
       </collision>
     </link>
-    <joint name="joint_right_leg_4" type="revolute">
+    <joint name="joint_right_leg_4" type="fixed">
       <origin xyz="0.2 0 -0.0514" rpy="0 0 0" />
       <parent link="right_leg_3" />

File: src/diablo_env_ros/urdf/robot.urdf (robot description, URDF)
Before this commit: robot diablo, 12 links, 11 joints
Links:
- link left_leg_4: geometry collision box size=0.0925 0.0925 0.0925; visual box size=0.0925 0.0925 0.0925
- link right_leg_4: geometry collision box size=0.0925 0.0925 0.0925; visual box size=0.0925 0.0925 0.0925

Commit message: changes the reward system and a2c code

File: src/diablo_env_ros/urdf/description.xacro (robot description, xacro)
@@ -352,5 +352,5 @@
       </collision>
     </link>
-    <joint name="joint_right_leg_4" type="fixed">
+    <joint name="joint_right_leg_4" type="revolute">
       <origin xyz="0.2 0 -0.0514" rpy="0 0 0" />
       <parent link="right_leg_3" />
