Commit message: amx torque was not enough

File: src/diablo_env_ros/urdf/description.xacro (robot description, xacro)
@@ -4,9 +4,4 @@
     <!-- <link name="world"/> -->
     <link name="base_footprint">
-      <inertial>
-        <mass value="0.0001"/>
-        <origin xyz="0 0 0" rpy="0 0 0"/>
-        <inertia ixx="1e-6" ixy="0" ixz="0" iyy="1e-6" iyz="0" izz="1e-6"/>
-      </inertial>
     </link>
     <link name="base_link">
@@ -26,6 +21,6 @@
         <origin xyz="0 0 0" rpy="0 0 0" />
         <geometry>
-          <sphere radius="0.15"/>
-          <!-- <box size="0.47 0.3 0.19"/> -->
+          <!-- <sphere radius="0.15"/> -->
+          <box size="0.4 0.3 0.19"/>
           <!-- <mesh filename="file://$(find diablo_env_ros)/meshes/base_link.STL" /> -->
         </geometry>
@@ -271,5 +266,5 @@
       <child link="right_leg_1" />
       <axis xyz="0 0 1" />
-      <limit lower="-0.1" upper="0.1" effort="100" velocity="100" />
+      <limit lower="-0.7854" upper="0.7854" effort="100" velocity="100" />
     </joint>
     <link name="right_leg_2">

File: src/diablo_env_ros/urdf/robot.urdf (robot description, URDF)
Before this commit: robot diablo, 12 links, 11 joints
Links:
- link base_footprint: mass 0.0001 -> None
- link base_link: geometry collision box size=0.4 0.3 0.19; visual mesh filename=file:///home/basanta-joshi/Desktop/virtual_environment/diab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
Joints:
- joint joint_right_leg_1: limit lower=-0.1 upper=0.1 effort=100 velocity=100 -> lower=-0.7854 upper=0.7854 effort=100 velocity=100

File: src/diablo_env_ros/urdf/robot.xacro (robot description, xacro)
@@ -107,5 +107,5 @@
   </gazebo>
   <gazebo reference="lidar_frame">
-    <sensor name='gpu_lidar' type='gpu_lidar'>"
+    <sensor name='gpu_lidar' type='gpu_lidar'>
         <pose relative_to='lidar_frame'>0 0 0 0 0 0</pose>
         <topic>lidar</topic>

Commit message: change simulation node rewards run rollout buffer

File: src/diablo_env_ros/urdf/description.xacro (robot description, xacro)
@@ -219,7 +219,7 @@
         <origin xyz="0 0 0" rpy="0 0 0" />
         <geometry>
-          <box size="0.0925 0.0925 0.0925"/>
+          <!-- <box size="0.0925 0.0925 0.0925"/> -->
           <!-- <cylinder length="0.034" radius="0.0925"/> -->
-          <!-- <mesh filename="file://$(find diablo_env_ros)/meshes/left_leg_4.STL" /> -->
+          <mesh filename="file://$(find diablo_env_ros)/meshes/left_leg_4.STL" />
         </geometry>
         <material name="silver"/>
@@ -228,6 +228,6 @@
         <origin xyz="0 0 0" rpy="0 0 0" />
         <geometry>
-          <box size="0.0925 0.0925 0.0925"/>
-          <!-- <cylinder length="0.034" radius="0.0925"/> -->
+          <!-- <box size="0.0925 0.0925 0.0925"/> -->
+          <cylinder length="0.034" radius="0.0925"/>
           <!-- <mesh filename="file://$(find diablo_env_ros)/meshes/left_leg_4.STL" /> -->
         </geometry>
@@ -238,5 +238,7 @@
       <parent link="left_leg_3" />
       <child link="left_leg_4" />
-      <axis xyz="0 0 1" />
+      <axis xyz="0 0 1" >
+        <dynamics damping="0.05" friction="0.01"/>
+      </axis>
       <limit lower="-6.283185e4" upper="6.283185e4" effort="100" velocity="100" />
     </joint>
@@ -333,6 +335,6 @@
         <origin xyz="0 0 0" rpy="0 0 0" />
         <geometry>
-          <box size="0.0925 0.0925 0.0925"/>
-          <!-- <mesh filename="file://$(find diablo_env_ros)/meshes/right_leg_4.STL" /> -->
+          <!-- <box size="0.0925 0.0925 0.0925"/> -->
+          <mesh filename="file://$(find diablo_env_ros)/meshes/right_leg_4.STL" />
         </geometry>
         <material name="silver"/>
@@ -341,6 +343,6 @@
         <origin xyz="0 0 0" rpy="0 0 0" />
         <geometry>
-          <box size="0.0925 0.0925 0.0925"/>
-          <!-- <cylinder length="0.034" radius="0.0925"/> -->
+          <!-- <box size="0.0925 0.0925 0.0925"/> -->
+          <cylinder length="0.034" radius="0.0925"/>
           <!-- <mesh filename="file://$(find diablo_env_ros)/meshes/right_leg_4.STL" /> -->
         </geometry>
@@ -351,5 +353,7 @@
       <parent link="right_leg_3" />
       <child link="right_leg_4" />
-      <axis xyz="0 0 1" />
+      <axis xyz="0 0 1" >
+        <dynamics damping="0.05" friction="0.01"/>
+      </axis>
       <limit lower="-6.283185e4" upper="6.283185e4" effort="100" velocity="100" />
     </joint>

File: src/diablo_env_ros/urdf/robot.urdf (robot description, URDF)
Before this commit: robot diablo, 12 links, 11 joints
Links:
- link left_leg_4: geometry collision cylinder length=0.034 radius=0.0925; visual mesh filename=file:///home/basanta-joshi/Desktop/virtual_environment/diab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
- link right_leg_4: geometry collision cylinder length=0.034 radius=0.0925; visual mesh filename=file:///home/basanta-joshi/Desktop/virtual_environment/diab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
