Commit message: adding some fixes in a2c

File: src/diablo_env_ros/urdf/description.xacro (robot description, xacro)
@@ -208,5 +208,5 @@
       <child link="left_leg_3" />
       <axis xyz="0 0 1" />
-      <limit lower="-2.670354" upper="-0.698132" effort="100" velocity="100" />
+      <limit lower="-2.670354" upper="0.2" effort="100" velocity="100" />
     </joint>
     <link name="left_leg_4">
@@ -324,5 +324,5 @@
       <child link="right_leg_3" />
       <axis xyz="0 0 1" />
-      <limit lower="-2.670354" upper="-0.698132" effort="100" velocity="100" />
+      <limit lower="-2.670354" upper="0.2" effort="100" velocity="100" />
     </joint>
     <link name="right_leg_4">

File: src/diablo_env_ros/urdf/robot.urdf (robot description, URDF)
Before this commit: robot diablo, 12 links, 11 joints
Joints:
- joint joint_left_leg_3: limit lower=-2.670354 upper=-0.698132 effort=100 velocity=100 -> lower=-2.670354 upper=0.2 effort=100 velocity=100
- joint joint_right_leg_3: limit lower=-2.670354 upper=-0.698132 effort=100 velocity=100 -> lower=-2.670354 upper=0.2 effort=100 velocity=100

File: src/diablo_env_ros/urdf/robot.xacro (robot description, xacro)
@@ -3,6 +3,4 @@
   <xacro:arg name="prefix" default="" />
   <xacro:arg name="use_tower" default="false" />
-  <xacro:property name="sim_env" value="$(arg sim_env)" />
-  <xacro:property name="ctrl_mode" value="$(arg ctrl_mode)" />
   <xacro:arg name="yaml_path" default="" />
   <xacro:include filename="$(find diablo_env_ros)/urdf/materials.xacro" />
@@ -131,3 +129,10 @@
     </sensor>
   </gazebo>
+  <gazebo>
+    <plugin filename="gz-sim-pose-publisher-system" name="gz::sim::systems::PosePublisher">
+      <publish_model_pose>true</publish_model_pose>
+      <publish_link_pose>false</publish_link_pose>
+      <use_pose_vector_msg>false</use_pose_vector_msg>
+    </plugin>
+  </gazebo>
 </robot>
